File: OpenHardwareExG_ActiveElectrode.kicad_pcb (KiCad board)
At the start: 4 copper layers, 19.3 x 19.3 mm, 13 parts, among them K1 CONN_3, P1 CONN_1, U1 LMP7715, U2 LMP7721

Commit message: CERN OHL v1.1 logo, and text
Parts:
- added G***: LOGO, LOGO, F.Cu at (103.6, 43.3)
Other:
- board text added: "CERN OHL v1.1"
- board text added: "OpenElectronicsLab Ace Medlock Eric Herman Kendrick Shaw"
- board text added: "OpenHardwareExG ActiveElectrode"
Changed lines of the file:
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@@
     (area 90.678 40.64 112.776001 62.230001)
     (thickness 1.6)
-    (drawings 1)
+    (drawings 4)
     (tracks 138)
     (zones 0)
-    (modules 13)
+    (modules 14)
     (nets 11)
   )
@@
     (pad_to_mask_clearance 0)
     (aux_axis_origin 0 0)
-    (visible_elements 7FFEFFFF)
+    (visible_elements 7FFEFBFF)
     (pcbplotparams
       (layerselection 0x00030_80000001)
@@
     (add_net GND)
   )
+  (module LOGO (layer F.Cu)
+    (at 103.6 43.3)
+    (fp_text reference G*** (at 0 1.59004) (layer F.SilkS) hide
+      (effects (font (size 0.13462 0.13462) (thickness 0.0254)))
+    )
+    (fp_text value LOGO (at 0 -1.59004) (layer F.SilkS) hide
+      (effects (font (size 0.13462 0.13462) (thickness 0.0254)))
+    )
+    (fp_poly (pts (xy -0.90932 1.3462) (xy -0.89154 1.33858) (xy -0.85852 1.31572) (xy -0.80772 1.2827)
+      (xy -0.7493 1.2446) (xy -0.68834 1.20396) (xy -0.64008 1.17094) (xy -0.60452 1.14808)
+      (xy -0.59182 1.14046) (xy -0.5842 1.143) (xy -0.55626 1.15824) (xy -0.51562 1.17856)
+      (xy -0.49022 1.19126) (xy -0.45212 1.2065) (xy -0.43434 1.21158) (xy -0.4318 1.2065)
+      (xy -0.41656 1.17602) (xy -0.39624 1.12776) (xy -0.3683 1.06172) (xy -0.33528 0.98552)
+      (xy -0.29972 0.90424) (xy -0.2667 0.82042) (xy -0.23368 0.74168) (xy -0.2032 0.66802)
+      (xy -0.18034 0.6096) (xy -0.1651 0.56896) (xy -0.15748 0.55118) (xy -0.16002 0.54864)
+      (xy -0.1778 0.53086) (xy -0.21082 0.50546) (xy -0.28194 0.44704) (xy -0.35306 0.36068)
+      (xy -0.39624 0.26162) (xy -0.40894 0.14986) (xy -0.39878 0.04826) (xy -0.35814 -0.04826)
+      (xy -0.28956 -0.13716) (xy -0.20574 -0.2032) (xy -0.10922 -0.24384) (xy 0 -0.25654)
+      (xy 0.10414 -0.24638) (xy 0.2032 -0.20574) (xy 0.2921 -0.1397) (xy 0.3302 -0.09652)
+      (xy 0.381 -0.00508) (xy 0.41148 0.0889) (xy 0.41402 0.11176) (xy 0.40894 0.21844)
+      (xy 0.37846 0.32004) (xy 0.32258 0.40894) (xy 0.24638 0.4826) (xy 0.23622 0.49022)
+      (xy 0.20066 0.51816) (xy 0.17526 0.53594) (xy 0.15748 0.55118) (xy 0.2921 0.87376)
+      (xy 0.31242 0.92456) (xy 0.35052 1.01346) (xy 0.381 1.08966) (xy 0.40894 1.15062)
+      (xy 0.42672 1.19126) (xy 0.43434 1.2065) (xy 0.43434 1.2065) (xy 0.44704 1.20904)
+      (xy 0.4699 1.20142) (xy 0.51562 1.17856) (xy 0.5461 1.16332) (xy 0.57912 1.14808)
+      (xy 0.59436 1.14046) (xy 0.6096 1.14808) (xy 0.64262 1.1684) (xy 0.68834 1.20142)
+      (xy 0.74676 1.23952) (xy 0.80264 1.27762) (xy 0.85344 1.31064) (xy 0.889 1.33604)
+      (xy 0.90678 1.34366) (xy 0.90932 1.34366) (xy 0.9271 1.33604) (xy 0.95504 1.31064)
+      (xy 0.99822 1.27) (xy 1.06172 1.20904) (xy 1.07188 1.19888) (xy 1.12268 1.14808)
+      (xy 1.16332 1.10236) (xy 1.19126 1.07188) (xy 1.20142 1.05918) (xy 1.20142 1.05918)
+      (xy 1.19126 1.0414) (xy 1.1684 1.0033) (xy 1.13538 0.9525) (xy 1.09474 0.89154)
+      (xy 0.98806 0.7366) (xy 1.04648 0.59182) (xy 1.06426 0.5461) (xy 1.08712 0.49022)
+      (xy 1.1049 0.45212) (xy 1.11252 0.43434) (xy 1.1303 0.42926) (xy 1.1684 0.4191)
+      (xy 1.22682 0.40894) (xy 1.29794 0.39624) (xy 1.36398 0.38354) (xy 1.4224 0.37084)
+      (xy 1.46558 0.36322) (xy 1.4859 0.36068) (xy 1.49098 0.3556) (xy 1.49352 0.34798)
+      (xy 1.49606 0.32766) (xy 1.4986 0.28956) (xy 1.4986 0.23368) (xy 1.4986 0.14986)
+      (xy 1.4986 0.14224) (xy 1.4986 0.0635) (xy 1.49606 0) (xy 1.49352 -0.0381)
+      (xy 1.49098 -0.05588) (xy 1.49098 -0.05588) (xy 1.4732 -0.06096) (xy 1.43002 -0.06858)
+      (xy 1.3716 -0.08128) (xy 1.30048 -0.09398) (xy 1.2954 -0.09398) (xy 1.22428 -0.10922)
+      (xy 1.16586 -0.12192) (xy 1.12268 -0.12954) (xy 1.1049 -0.13716) (xy 1.10236 -0.14224)
+      (xy 1.08712 -0.17018) (xy 1.0668 -0.21336) (xy 1.04394 -0.2667) (xy 1.02108 -0.32258)
+      (xy 1.00076 -0.37338) (xy 0.98806 -0.40894) (xy 0.98298 -0.42672) (xy 0.98298 -0.42672)
+      (xy 0.99314 -0.4445) (xy 1.01854 -0.48006) (xy 1.0541 -0.53086) (xy 1.09474 -0.59182)
+      (xy 1.09728 -0.5969) (xy 1.13792 -0.65786) (xy 1.17094 -0.70866) (xy 1.1938 -0.74422)
+      (xy 1.20142 -0.75946) (xy 1.20142 -0.762) (xy 1.18872 -0.77978) (xy 1.15824 -0.8128)
+      (xy 1.11252 -0.85852) (xy 1.06172 -0.91186) (xy 1.04394 -0.9271) (xy 0.98552 -0.98552)
+      (xy 0.94488 -1.02108) (xy 0.91948 -1.0414) (xy 0.90932 -1.04648) (xy 0.90678 -1.04648)
+      (xy 0.889 -1.03632) (xy 0.8509 -1.01092) (xy 0.8001 -0.97536) (xy 0.73914 -0.93472)
+      (xy 0.7366 -0.93218) (xy 0.67564 -0.89154) (xy 0.62484 -0.85598) (xy 0.58928 -0.83312)
+      (xy 0.57404 -0.8255) (xy 0.5715 -0.8255) (xy 0.54864 -0.83058) (xy 0.50546 -0.84582)
+      (xy 0.45212 -0.86614) (xy 0.39624 -0.889) (xy 0.34544 -0.90932) (xy 0.30988 -0.9271)
+      (xy 0.2921 -0.93726) (xy 0.28956 -0.93726) (xy 0.28448 -0.96012) (xy 0.27432 -1.00584)
+      (xy 0.26162 -1.0668) (xy 0.24638 -1.14046) (xy 0.24384 -1.15062) (xy 0.23114 -1.22428)
+      (xy 0.22098 -1.2827) (xy 0.21082 -1.32334) (xy 0.20828 -1.34112) (xy 0.19812 -1.34112)
+      (xy 0.16256 -1.34366) (xy 0.10922 -1.3462) (xy 0.04318 -1.3462) (xy -0.02286 -1.3462)
+      (xy -0.0889 -1.3462) (xy -0.14478 -1.34366) (xy -0.18542 -1.34112) (xy -0.2032 -1.33604)
+      (xy -0.2032 -1.33604) (xy -0.20828 -1.31318) (xy -0.21844 -1.27) (xy -0.23114 -1.2065)
+      (xy -0.24638 -1.13284) (xy -0.24892 -1.12014) (xy -0.26162 -1.04902) (xy -0.27432 -0.9906)
+      (xy -0.28194 -0.94996) (xy -0.28702 -0.93472) (xy -0.2921 -0.93218) (xy -0.32258 -0.91694)
+      (xy -0.37084 -0.89916) (xy -0.42926 -0.87376) (xy -0.56642 -0.81788) (xy -0.73406 -0.93472)
+      (xy -0.7493 -0.94488) (xy -0.81026 -0.98552) (xy -0.86106 -1.01854) (xy -0.89662 -1.0414)
+      (xy -0.90932 -1.04902) (xy -0.91186 -1.04902) (xy -0.9271 -1.03378) (xy -0.96012 -1.0033)
+      (xy -1.00584 -0.95758) (xy -1.05918 -0.90678) (xy -1.09982 -0.86614) (xy -1.14554 -0.82042)
+      (xy -1.17348 -0.7874) (xy -1.19126 -0.76708) (xy -1.19634 -0.75438) (xy -1.1938 -0.74676)
+      (xy -1.18364 -0.72898) (xy -1.15824 -0.69342) (xy -1.12522 -0.64008) (xy -1.08458 -0.58166)
+      (xy -1.04902 -0.53086) (xy -1.01346 -0.47498) (xy -0.9906 -0.43434) (xy -0.98044 -0.41656)
+      (xy -0.98298 -0.4064) (xy -0.99568 -0.37338) (xy -1.016 -0.32512) (xy -1.0414 -0.26416)
+      (xy -1.09982 -0.13208) (xy -1.18618 -0.1143) (xy -1.23952 -0.10414) (xy -1.31318 -0.09144)
+      (xy -1.3843 -0.0762) (xy -1.49606 -0.05588) (xy -1.4986 0.34798) (xy -1.48082 0.3556)
+      (xy -1.46558 0.36068) (xy -1.42494 0.37084) (xy -1.36652 0.381) (xy -1.29794 0.3937)
+      (xy -1.23698 0.4064) (xy -1.17856 0.41656) (xy -1.13538 0.42418) (xy -1.1176 0.42926)
+      (xy -1.11252 0.43434) (xy -1.09728 0.46482) (xy -1.07696 0.51054) (xy -1.0541 0.56388)
+      (xy -1.0287 0.6223) (xy -1.00838 0.6731) (xy -0.99314 0.71374) (xy -0.98806 0.73406)
+      (xy -0.99568 0.7493) (xy -1.01854 0.78486) (xy -1.05156 0.83566) (xy -1.0922 0.89408)
+      (xy -1.13284 0.9525) (xy -1.16586 1.0033) (xy -1.19126 1.03886) (xy -1.19888 1.05664)
+      (xy -1.1938 1.0668) (xy -1.17094 1.09474) (xy -1.12776 1.14046) (xy -1.06172 1.2065)
+      (xy -1.04902 1.21666) (xy -0.99822 1.26746) (xy -0.9525 1.3081) (xy -0.92202 1.33604)
+      (xy -0.90932 1.3462)) (layer F.SilkS) (width 0.00254))
+  )
   (module Capacitors_SMD:C_0201 (layer F.Cu)
     (at 97.79 57.785)
@@
     (tags "capacitor 0402")
     (attr smd)
-    (fp_text reference C2 (at -1.778 -0.0254 270) (layer F.SilkS)
+    (fp_text reference C2 (at -0.915 -1.17 360) (layer F.SilkS)
       (effects (font (size 0.6 0.6) (thickness 0.127)))
     )
@@
     (tags "resistor 0402")
     (attr smd)
-    (fp_text reference R2 (at 0.8382 -1.0668) (layer F.SilkS)
+    (fp_text reference R2 (at -1.225 -0.98) (layer F.SilkS)
       (effects (font (size 0.6 0.6) (thickness 0.127)))
     )
@@
     )
   )
+  (gr_text "OpenElectronicsLab\nAce Medlock\nEric Herman\nKendrick Shaw" (at 106 49.4) (layer F.SilkS)
+    (effects (font (size 0.5 0.5) (thickness 0.1)))
+  )
+  (gr_text "OpenHardwareExG\nActiveElectrode" (at 100 51.1 90) (layer F.SilkS)
+    (effects (font (size 0.6 0.6) (thickness 0.127)))
+  )
+  (gr_text "CERN OHL\nv1.1" (at 104 45.7) (layer F.SilkS)
+    (effects (font (size 0.6 0.6) (thickness 0.127)))
+  )
   (gr_circle (center 101.5492 51.181) (end 101.5492 60.833) (layer Edge.Cuts) (width 0.1))
